Commit message: feat: add gazebo robot

File: src/urdf_tutorial/urdf/robot_3.xacro (robot description, xacro)
@@ -30,4 +30,13 @@
             <material name="white"/>
         </visual>
+        <collision>
+            <origin xyz="0.1 0 0.03"/>
+            <geometry>
+                <box size="0.2 0.1 0.06"/>
+            </geometry>
+        </collision>
+        <xacro:inertial_box mass="0.5" x="0.2" y="0.1" z="0.06">
+            <origin xyz="0.1 0 0.03" rpy="0 0 0"/>
+        </xacro:inertial_box>
     </link>
     <!-- LEFT WHEEL LINK -->
@@ -54,4 +63,7 @@
         </xacro:inertial_cylinder>
     </link>
+    <gazebo reference="left_wheel">
+        <material>Gazebo/Black</material>
+    </gazebo>
     <!-- RIGHT WHEEL LINK -->
     <joint name="right_wheel_joint" type="continuous">
@@ -77,4 +89,7 @@
         </xacro:inertial_cylinder>
     </link>
+    <gazebo reference="right_wheel">
+        <material>Gazebo/Black</material>
+    </gazebo>
     <!-- CASTER WHEEL LINK -->
     <joint name="caster_wheel_joint" type="fixed">
@@ -99,3 +114,10 @@
         </xacro:inertial_sphere>
     </link>
+    <gazebo reference="caster_wheel">
+        <material>Gazebo/Blue</material>
+        <mu1 value="0.001"/>
+        <mu2 value="0.001"/>
+    </gazebo>
+    <!-- GAZEBO -->
+    <xacro:include filename="gazebo.xacro"/>
 </robot>
